File: haku.kicad_pcb (KiCad board)
At the start: 2 copper layers, 323.9 x 97 mm, 180 parts, among them SW1 SW_Push, U1 ATmega32U4-AU, U2 SRV05-4, Y1 16MHz

Commit message: some finishing touches
Parts:
- removed the G*** at (52.7, 180.0)
- added G***: LOGO, board_logos:designed-by1, F.Cu at (62.7, 178.6)

Commit message: final changes before protos
Parts:
- added C15: 0.1uF, Capacitor_SMD:C_0805_2012Metric, B.Cu at (338.2, 133.9)
- added G***: LOGO, board_logos:prototype, B.Cu at (77.0, 123.8)
- moved U2 5.21 mm to (105.2, 97.5)
- moved F1 4.96 mm to (103.1, 103.1)
- moved C10 2.79 mm to (338.2, 102.4), turned to 0 degrees
- moved C14 2.73 mm to (338.2, 127.8), turned to 0 degrees
- moved C12 2.68 mm to (338.2, 115.1), turned to 0 degrees
- moved C11 2.68 mm to (338.2, 108.7), turned to 0 degrees
- moved C13 2.68 mm to (338.2, 121.4), turned to 0 degrees
- moved C9 2.58 mm to (338.2, 96.0), turned to 0 degrees
Connections:
- U2 pad 5: +5V -> VCC
Routing:
- net +5V: track 513.0 -> 488.5 mm, vias 21 -> 23
- net VCC: track 4.66 -> 10.5 mm
- net GND: track 146.0 -> 144.1 mm
