File: haku.sch (KiCad schematic (older format))
At the start: 172 parts, among them SW1 SW_Push, U1 ATmega32U4-AU, U2 SRV05-4, Y1 16MHz

Commit message: lots of changes
Parts:
- added C10, C11, C12, C13, C14, C9: 0.1uF, Capacitor_SMD:C_0805_2012Metric, symbol Device:C_Small
Connections:
- net +5V: now also C10.1, C11.1, C12.1, C13.1, C14.1, C9.1
- net GND: now also C10.2, C11.2, C12.2, C13.2, C14.2, C9.2
Changed lines of the file:
@@
 Text GLabel 5100 2100 2    50   Input ~ 0
 IND_LED2
+$Comp
+L Device:C_Small C9
+U 1 1 5EA86DAC
+P 950 5450
+F 0 "C9" H 1042 5496 50  0000 L CNN
+F 1 "0.1uF" H 1042 5405 50  0000 L CNN
+F 2 "Capacitor_SMD:C_0805_2012Metric" H 950 5450 50  0001 C CNN
+F 3 "~" H 950 5450 50  0001 C CNN
+	1    950  5450
+	1    0    0    -1
+$EndComp
+$Comp
+L Device:C_Small C10
+U 1 1 5EA86DB6
+P 1350 5450
+F 0 "C10" H 1442 5496 50  0000 L CNN
+F 1 "0.1uF" H 1442 5405 50  0000 L CNN
+F 2 "Capacitor_SMD:C_0805_2012Metric" H 1350 5450 50  0001 C CNN
+F 3 "~" H 1350 5450 50  0001 C CNN
+	1    1350 5450
+	1    0    0    -1
+$EndComp
+$Comp
+L Device:C_Small C11
+U 1 1 5EA86DC0
+P 1750 5450
+F 0 "C11" H 1842 5496 50  0000 L CNN
+F 1 "0.1uF" H 1842 5405 50  0000 L CNN
+F 2 "Capacitor_SMD:C_0805_2012Metric" H 1750 5450 50  0001 C CNN
+F 3 "~" H 1750 5450 50  0001 C CNN
+	1    1750 5450
+	1    0    0    -1
+$EndComp
+Wire Wire Line
+	950  5350 1350 5350
+Connection ~ 1350 5350
+Wire Wire Line
+	1350 5350 1750 5350
+Connection ~ 1750 5350
+Wire Wire Line
+	1750 5350 1950 5350
+Connection ~ 1350 5550
+Wire Wire Line
+	1350 5550 950  5550
+Connection ~ 1750 5550
+Wire Wire Line
+	1750 5550 1350 5550
+Wire Wire Line
+	2150 5550 1950 5550
+Wire Wire Line
+	1950 5550 1950 5650
+Wire Wire Line
+	1950 5350 1950 5250
+$Comp
+L power:+5V #PWR0123
+U 1 1 5EA86DD6
+P 1950 5250
+F 0 "#PWR0123" H 1950 5100 50  0001 C CNN
+F 1 "+5V" H 1965 5423 50  0000 C CNN
+F 2 "" H 1950 5250 50  0001 C CNN
+F 3 "" H 1950 5250 50  0001 C CNN
+	1    1950 5250
+	1    0    0    -1
+$EndComp
+$Comp
+L power:GND #PWR0124
+U 1 1 5EA86DE0
+P 1950 5650
+F 0 "#PWR0124" H 1950 5400 50  0001 C CNN
+F 1 "GND" H 1955 5477 50  0000 C CNN
+F 2 "" H 1950 5650 50  0001 C CNN
+F 3 "" H 1950 5650 50  0001 C CNN
+	1    1950 5650
+	1    0    0    -1
+$EndComp
+$Comp
+L Device:C_Small C12
+U 1 1 5EAD03DB
+P 2150 5450
+F 0 "C12" H 2242 5496 50  0000 L CNN
+F 1 "0.1uF" H 2242 5405 50  0000 L CNN
+F 2 "Capacitor_SMD:C_0805_2012Metric" H 2150 5450 50  0001 C CNN
+F 3 "~" H 2150 5450 50  0001 C CNN
+	1    2150 5450
+	1    0    0    -1
+$EndComp
+$Comp
+L Device:C_Small C13
+U 1 1 5EAD03E5
+P 2550 5450
+F 0 "C13" H 2642 5496 50  0000 L CNN
+F 1 "0.1uF" H 2642 5405 50  0000 L CNN
+F 2 "Capacitor_SMD:C_0805_2012Metric" H 2550 5450 50  0001 C CNN
+F 3 "~" H 2550 5450 50  0001 C CNN
+	1    2550 5450
+	1    0    0    -1
+$EndComp
+$Comp
+L Device:C_Small C14
+U 1 1 5EAD03EF
+P 2950 5450
+F 0 "C14" H 3042 5496 50  0000 L CNN
+F 1 "0.1uF" H 3042 5405 50  0000 L CNN
+F 2 "Capacitor_SMD:C_0805_2012Metric" H 2950 5450 50  0001 C CNN
+F 3 "~" H 2950 5450 50  0001 C CNN
+	1    2950 5450
+	1    0    0    -1
+$EndComp
+Wire Wire Line
+	2150 5350 2550 5350
+Connection ~ 2550 5350
+Wire Wire Line
+	2550 5350 2950 5350
+Connection ~ 2550 5550
+Wire Wire Line
+	2550 5550 2150 5550
+Wire Wire Line
+	2950 5550 2550 5550
+Connection ~ 2150 5350
+Connection ~ 2150 5550
+Connection ~ 1950 5550
+Wire Wire Line
+	1950 5550 1750 5550
+Connection ~ 1950 5350
+Wire Wire Line
+	1950 5350 2150 5350
 $EndSCHEMATC

Commit message: final changes before protos
Parts:
- added C15: 0.1uF, Capacitor_SMD:C_0805_2012Metric, symbol Device:C_Small
Connections:
- net +5V: now also C15.1; no longer U2.5 (VP)
- net GND: now also C15.2
- net VCC: now also U2.5 (VP)
Changed lines of the file:
@@
-	1    0    0    -1
-$EndComp
-$Comp
-L power:+5V #PWR0117
-U 1 1 5E920182
-P 9150 1350
-F 0 "#PWR0117" H 9150 1200 50  0001 C CNN
-F 1 "+5V" H 9165 1523 50  0000 C CNN
-F 2 "" H 9150 1350 50  0001 C CNN
-F 3 "" H 9150 1350 50  0001 C CNN
-	1    9150 1350
 	1    0    0    -1
 $EndComp
@@
 	1350 5350 1750 5350
 Connection ~ 1750 5350
-Wire Wire Line
-	1750 5350 1950 5350
 Connection ~ 1350 5550
 Wire Wire Line
@@
 	1750 5550 1350 5550
 Wire Wire Line
-	2150 5550 1950 5550
-Wire Wire Line
-	1950 5550 1950 5650
-Wire Wire Line
-	1950 5350 1950 5250
+	2150 5550 2150 5650
+Wire Wire Line
+	2150 5350 2150 5250
 $Comp
 L power:+5V #PWR0123
 U 1 1 5EA86DD6
-P 1950 5250
-F 0 "#PWR0123" H 1950 5100 50  0001 C CNN
-F 1 "+5V" H 1965 5423 50  0000 C CNN
-F 2 "" H 1950 5250 50  0001 C CNN
-F 3 "" H 1950 5250 50  0001 C CNN
-	1    1950 5250
+P 2150 5250
+F 0 "#PWR0123" H 2150 5100 50  0001 C CNN
+F 1 "+5V" H 2165 5423 50  0000 C CNN
+F 2 "" H 2150 5250 50  0001 C CNN
+F 3 "" H 2150 5250 50  0001 C CNN
+	1    2150 5250
 	1    0    0    -1
 $EndComp
@@
 L power:GND #PWR0124
 U 1 1 5EA86DE0
-P 1950 5650
-F 0 "#PWR0124" H 1950 5400 50  0001 C CNN
-F 1 "GND" H 1955 5477 50  0000 C CNN
-F 2 "" H 1950 5650 50  0001 C CNN
-F 3 "" H 1950 5650 50  0001 C CNN
-	1    1950 5650
+P 2150 5650
+F 0 "#PWR0124" H 2150 5400 50  0001 C CNN
+F 1 "GND" H 2155 5477 50  0000 C CNN
+F 2 "" H 2150 5650 50  0001 C CNN
+F 3 "" H 2150 5650 50  0001 C CNN
+	1    2150 5650
 	1    0    0    -1
 $EndComp
@@
 Connection ~ 2150 5350
 Connection ~ 2150 5550
-Connection ~ 1950 5550
-Wire Wire Line
-	1950 5550 1750 5550
-Connection ~ 1950 5350
-Wire Wire Line
-	1950 5350 2150 5350
+$Comp
+L Device:C_Small C15
+U 1 1 5EB1DFFE
+P 3350 5450
+F 0 "C15" H 3442 5496 50  0000 L CNN
+F 1 "0.1uF" H 3442 5405 50  0000 L CNN
+F 2 "Capacitor_SMD:C_0805_2012Metric" H 3350 5450 50  0001 C CNN
+F 3 "~" H 3350 5450 50  0001 C CNN
+	1    3350 5450
+	1    0    0    -1
+$EndComp
+Wire Wire Line
+	2950 5350 3350 5350
+Wire Wire Line
+	3350 5550 2950 5550
+Connection ~ 2950 5350
+Connection ~ 2950 5550
+Wire Wire Line
+	1750 5550 2150 5550
+Wire Wire Line
+	1750 5350 2150 5350
+$Comp
+L power:VCC #PWR?
+U 1 1 5ED3BF2B
+P 9150 1350
+F 0 "#PWR?" H 9150 1200 50  0001 C CNN
+F 1 "VCC" H 9150 1500 50  0000 C CNN
+F 2 "" H 9150 1350 50  0001 C CNN
+F 3 "" H 9150 1350 50  0001 C CNN
+	1    9150 1350
+	1    0    0    -1
+$EndComp
 $EndSCHEMATC
